Commit message: cosmetics

File: description/face.xacro (robot description, xacro)
@@ -10,5 +10,5 @@
             <origin xyz="0 0.05 0.01" rpy="0 ${pi/2} 0"/>
             <geometry>
-                <cylinder radius="0.01" length="0.002"/>
+                <cylinder radius="0.005" length="0.002"/>
             </geometry>
             <material name="black"/>
@@ -17,5 +17,5 @@
             <origin xyz="0 -0.05 0.01" rpy="0 ${pi/2} 0"/>
             <geometry>
-                <cylinder radius="0.01" length="0.002"/>
+                <cylinder radius="0.005" length="0.002"/>
             </geometry>
             <material name="black"/>

File: description/lidar.xacro (robot description, xacro)
@@ -4,5 +4,5 @@
         <parent link="chassis"/>
         <child link="laser_frame"/>
-        <origin xyz="0.122 0 0.212" rpy="0 0 0"/>
+        <origin xyz="0.122 0 0.112" rpy="0 0 0"/>
     </joint>
     <link name="laser_frame">
@@ -11,12 +11,5 @@
                 <cylinder radius="0.05" length="0.04"/>
             </geometry>
-            <material name="black"/>
-        </visual>
-        <visual>
-            <origin xyz="0 0 -0.05"/>
-            <geometry>
-                <cylinder radius="0.01" length="0.1"/>
-            </geometry>
-            <material name="black"/>
+            <material name="blue"/>
         </visual>
         <collision>
@@ -30,5 +23,5 @@
     </link>
     <gazebo reference="laser_frame">
-        <material>Gazebo/Black</material>
+        <material>Gazebo/Blue</material>
         <sensor name="laser" type="ray">
             <pose> 0 0 0 0 0 0 </pose>
