Commit message: changed face.xacro

File: description/camera.xacro (robot description, xacro)
@@ -4,5 +4,5 @@
         <parent link="chassis"/>
         <child link="camera_link"/>
-        <origin xyz="0.276 0 0.181" rpy="0 0.18 0"/>
+        <origin xyz="0.3 0 0.12" rpy="0 0 0"/>
     </joint>
     <link name="camera_link">
@@ -10,11 +10,4 @@
             <geometry>
                 <box size="0.010 0.03 0.03"/>
-            </geometry>
-            <material name="black"/>
-        </visual>
-        <visual>
-            <origin xyz="0 0 -0.05"/>
-            <geometry>
-                <cylinder radius="0.002" length="0.1"/>
             </geometry>
             <material name="black"/>
@@ -34,5 +27,5 @@
             <update_rate>10</update_rate>
             <camera>
-                <horizontal_fov>1.089</horizontal_fov>
+                <horizontal_fov>1.15192</horizontal_fov>
                 <image>
                     <format>R8G8B8</format>

File: description/face.xacro (robot description, xacro)
@@ -8,14 +8,14 @@
     <link name="face_link">
         <visual>
-            <origin xyz="0 0.05 0.01" rpy="0 ${pi/2} 0"/>
+            <origin xyz="0 0.025 0.01" rpy="0 ${pi/2} 0"/>
             <geometry>
-                <cylinder radius="0.005" length="0.002"/>
+                <cylinder radius="0.01" length="0.002"/>
             </geometry>
             <material name="black"/>
         </visual>
         <visual>
-            <origin xyz="0 -0.05 0.01" rpy="0 ${pi/2} 0"/>
+            <origin xyz="0 -0.025 0.01" rpy="0 ${pi/2} 0"/>
             <geometry>
-                <cylinder radius="0.005" length="0.002"/>
+                <cylinder radius="0.01" length="0.002"/>
             </geometry>
             <material name="black"/>
@@ -24,5 +24,5 @@
             <origin xyz="-0.011 0 -0.00" rpy="0 ${1.5} 0"/>
             <geometry>
-                <cylinder radius="0.05" length="0.02"/>
+                <cylinder radius="0.025" length="0.02"/>
             </geometry>
             <material name="red"/>

File: description/gazebo_control.xacro (robot description, xacro)
@@ -6,6 +6,6 @@
             <left_joint>left_wheel_joint</left_joint>
             <right_joint>right_wheel_joint</right_joint>
-            <wheel_separation>0.297</wheel_separation>
-            <wheel_diameter>0.066</wheel_diameter>
+            <wheel_separation>0.200</wheel_separation>
+            <wheel_diameter>0.070</wheel_diameter>
             <!-- Limits -->
             <max_wheel_torque>200</max_wheel_torque>

File: description/lidar.xacro (robot description, xacro)
@@ -26,5 +26,5 @@
         <sensor name="laser" type="ray">
             <pose> 0 0 0 0 0 0 </pose>
-            <visualize>false</visualize>
+            <visualize>true</visualize>
             <update_rate>10</update_rate>
             <ray>
@@ -41,5 +41,5 @@
                 </range>
             </ray>
-            <plugin name="laser_controller" filename="libgazebo_ros_ray_sensor.so">
+            <plugin name="laser_controller" filename="libgazebo_ros_laser.so">
                 <ros>
                     <argument>~/out:=scan</argument>
